File: PCB/HackPad v3.kicad_sch (KiCad schematic)
At the start: 74 parts, among them Q1 BSS138, SW1 SW_MEC_5G, SW10 SW_MEC_5G, SW11 SW_MEC_5G, SW12 SW_MEC_5G, SW13 SW_MEC_5G, SW14 SW_MEC_5G, SW15 SW_MEC_5G, SW16 SW_MEC_5G, SW2 SW_MEC_5G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

Commit message: Update PCB and Gerber
Parts:
- U1: footprint Module:MOUDLE14P-XIAO-DIP-SMD -> Seeed Studio Xiao:XIAO-RP2040-DIP
- U2: symbol Interface_Expansion:MCP23017_SS -> Interface_Expansion:MCP23017_SO
Changed lines of the file:
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@@
 			)
 		)
-		(property "Footprint" "Module:MOUDLE14P-XIAO-DIP-SMD"
+		(property "Footprint" "Seeed Studio Xiao:XIAO-RP2040-DIP"
 			(at 135.128 69.088 0)
 			(effects
@@
 	)
 	(symbol
-		(lib_id "Interface_Expansion:MCP23017_SS")
+		(lib_id "Interface_Expansion:MCP23017_SO")
 		(at 149.86 168.91 0)
 		(unit 1)
