File: PCB/HackPad v3.kicad_pcb (KiCad board)
At the start: 2 copper layers, 76.7 x 100.7 mm, 78 parts, among them Q1 BSS138, SW1 SW_MEC_5G, SW10 SW_MEC_5G, SW11 SW_MEC_5G, SW12 SW_MEC_5G, SW13 SW_MEC_5G, SW14 SW_MEC_5G, SW15 SW_MEC_5G, SW16 SW_MEC_5G, SW2 SW_MEC_5G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

Commit message: Update PCB and Gerber
Parts:
- removed the H at (178.2, 145.0)
- removed the H at (105.7, 145.0)
Routing:
- net Net-(LEDD13-DOUT): track 33.2 -> 44.8 mm, vias 2 -> 4
- net GND: track 568.5 -> 558.8 mm
- net A2: track 45.7 -> 43.2 mm, vias 2 -> 4
- net VBUS: track 418.5 -> 419.6 mm
- net Net-(LEDD15-DOUT): track 32.6 -> 33.6 mm
- net Net-(LEDD14-DOUT): track 30.1 -> 30.9 mm
Other:
- board size 76.7 x 100.7 mm -> 76.7 x 98.7 mm

Commit message: Update files
Routing:
- net GND: track 558.8 -> 552.4 mm, vias 14 -> 13
- net S2: track 31.8 -> 34.9 mm, vias 1 -> 3
- net RGB: track 63.2 -> 62.3 mm, vias 7 -> 4
- net Net-(LEDD14-DOUT): track 30.9 -> 31.7 mm
- net Net-(LEDD15-DOUT): vias 4 -> 2

Commit message: Change PCB and Gerber
Routing:
- net C3: track 95.9 -> 95.0 mm
Changed lines of the file:
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@@
 	)
 	(segment
-		(start 128.9 55.1)
-		(end 128.9 55.9713)
+		(start 111.8585 54.5958)
+		(end 111.8585 55.8826)
 		(width 0.2)
 		(layer "B.Cu")
@@
 	)
 	(segment
-		(start 111.8585 54.5958)
-		(end 111.8585 55.8826)
+		(start 128.9 55.1)
+		(end 128.9 56.3)
 		(width 0.2)
 		(layer "B.Cu")
@@
 	)
 	(segment
-		(start 128.9 55.9713)
-		(end 130.8811 57.9524)
+		(start 112.8618 53.5925)
+		(end 111.8585 54.5958)
 		(width 0.2)
 		(layer "B.Cu")
@@
 	)
 	(segment
-		(start 130.8811 57.9524)
+		(start 130.5524 57.9524)
 		(end 142.088 57.9524)
 		(width 0.2)
@@
 	)
 	(segment
-		(start 112.8618 53.5925)
-		(end 111.8585 54.5958)
-		(width 0.2)
-		(layer "B.Cu")
-		(net 5)
-	)
-	(segment
 		(start 142.088 57.9524)
 		(end 156.9431 57.9524)
@@
 	)
 	(segment
+		(start 128.9 56.3)
+		(end 130.5524 57.9524)
+		(width 0.2)
+		(layer "B.Cu")
+		(net 5)
+	)
+	(segment
 		(start 157.3433 57.5522)
 		(end 160.4578 57.5522)
@@
 	)
 	(segment
-		(start 145.3681 46.8766)
-		(end 145.2148 46.7233)
-		(width 0.2)
-		(layer "F.Cu")
-		(net 10)
-	)
-	(segment
-		(start 140.625 47.9)
-		(end 140.625 46.7233)
-		(width 0.2)
-		(layer "F.Cu")
-		(net 10)
-	)
-	(segment
 		(start 124.0682 50.5336)
 		(end 123.7 50.9018)
@@
 	)
 	(segment
-		(start 145.2148 46.7233)
-		(end 140.625 46.7233)
+		(start 140.625 47.9)
+		(end 140.625 46.95)
 		(width 0.2)
 		(layer "F.Cu")
 		(net 10)
 	)
-	(via
-		(at 124.0682 50.5336)
-		(size 0.6)
-		(drill 0.3)
+	(via micro
+		(at 140.625 46.95)
+		(size 0.3)
+		(drill 0.1)
 		(layers "F.Cu" "B.Cu")
 		(net 10)
 	)
 	(via
-		(at 145.3681 46.8766)
+		(at 124.0682 50.5336)
 		(size 0.6)
 		(drill 0.3)
@@
 	)
 	(segment
+		(start 145.3681 47.9535)
+		(end 148.1199 50.7053)
+		(width 0.2)
+		(layer "B.Cu")
+		(net 10)
+	)
+	(segment
 		(start 168.1 55.11)
 		(end 169.1628 54.0472)
@@
 	)
 	(segment
+		(start 140.625 46.95)
+		(end 141.6285 47.9535)
+		(width 0.2)
+		(layer "B.Cu")
+		(net 10)
+	)
+	(segment
 		(start 114.4058 53.9942)
 		(end 113.3 55.1)
@@
 	)
 	(segment
-		(start 148.1199 50.7053)
+		(start 141.6285 47.9535)
 		(end 145.3681 47.9535)
 		(width 0.2)
@@
 	)
 	(segment
-		(start 145.3681 47.9535)
-		(end 145.3681 46.8766)
-		(width 0.2)
-		(layer "B.Cu")
-		(net 10)
-	)
-	(segment
 		(start 172.9112 53.4684)
 		(end 172.9112 52.932)
@@
 	)
 	(segment
-		(start 122.0846 89.0328)
-		(end 122.0846 89.0346)
-		(width 0.2)
-		(layer "F.Cu")
-		(net 13)
-	)
-	(segment
 		(start 121.9719 81.3466)
 		(end 121.9719 84.0744)
@@
 	)
 	(segment
-		(start 126.1746 88.6316)
-		(end 126.1716 88.6316)
-		(width 0.2)
-		(layer "F.Cu")
-		(net 29)
-	)
-	(segment
 		(start 125.5876 100.3951)
 		(end 126.1746 100.9821)
@@
 	)
 	(segment
-		(start 121.88 132.5)
-		(end 121.88 132.47)
-		(width 0.2)
-		(layer "F.Cu")
-		(net 38)
-	)
-	(segment
 		(start 137.61 139.455184)
 		(end 129.374816 131.22)
@@
 	(segment
 		(start 137.61 141.66)
-		(end 137.61 140.07)
-		(width 0.2)
-		(layer "F.Cu")
-		(net 38)
-	)
-	(segment
-		(start 137.61 140.07)
 		(end 137.61 139.455184)
 		(width 0.2)
@@
 	)
 	(segment
-		(start 135.082599 143.099999)
-		(end 134.8913 142.9087)
-		(width 0.2)
-		(layer "B.Cu")
-		(net 38)
-	)
-	(segment
 		(start 136.24 143.03)
 		(end 135.86 143.03)
@@
 	)
 	(segment
-		(start 145.54 49.646449)
+		(start 145.503551 49.646449)
 		(end 146.153551 49.646449)
 		(width 0.2)
@@
 	)
 	(segment
-		(start 145.54 49.646449)
-		(end 145.503551 49.646449)
-		(width 0.2)
-		(layer "F.Cu")
-		(net 42)
-	)
-	(segment
 		(start 173.5 55.2)
 		(end 173.7 55)
@@
 		(net 46)
 	)
-	(segment
-		(start 151.5535 62.5864)
-		(end 151.5836 62.5864)
-		(width 0.2)
-		(layer "F.Cu")
-		(net 46)
-	)
 	(via
 		(at 151.5535 62.5864)
@@
 	)
 	(segment
-		(start 136.725 51.249943)
-		(end 136.726 51.248943)
-		(width 0.2)
-		(layer "F.Cu")
-		(net 47)
-	)
-	(segment
 		(start 129.7924 64.6115)
 		(end 131.2982 66.1173)
@@
 	)
 	(segment
-		(start 136.725 51.475)
-		(end 136.725 51.249943)
-		(width 0.2)
-		(layer "F.Cu")
-		(net 47)
-	)
-	(segment
 		(start 129.7924 57.97719)
 		(end 129.7924 64.6115)
@@
 	(segment
 		(start 136.726 52.154)
-		(end 136.726 51.17)
+		(end 136.726 50.751057)
 		(width 0.2)
 		(layer "F.Cu")
@@
 		(width 0.2)
 		(layer "F.Cu")
-		(net 47)
-	)
-	(segment
-		(start 131.2982 66.1173)
-		(end 131.2927 66.1173)
-		(width 0.2)
-		(layer "F.Cu")
-		(net 47)
-	)
-	(segment
-		(start 136.726 51.248943)
-		(end 136.726 51.17)
-		(width 0.2)
-		(layer "F.Cu")
-		(net 47)
-	)
-	(segment
-		(start 136.726 51.17)
-		(end 136.726 50.751057)
-		(width 0.2)
-		(layer "F.Cu")
